File: KiCAD Stuff/stm32 external storage.sch (KiCad schematic (older format))
At the start: 0 parts

Commit message: made kicad footprints for INA239 and microsd
Parts:
- added J?: Micro_SD_Card_Adafruit, symbol micro_sd_card_adafruit:Micro_SD_Card_Adafruit
- added U?: STM32F407VGTx, Package_QFP:LQFP-100_14x14mm_P0.5mm, symbol MCU_ST_STM32F4:STM32F407VGTx
- added U?: INA239-Q1, symbol ina239-q1:INA239-Q1
Changed lines of the file:
@@
 Comment4 ""
 $EndDescr
+$Comp
+L MCU_ST_STM32F4:STM32F407VGTx U?
+U 1 1 614FFDC2
+P 2650 3800
+F 0 "U?" H 2650 911 50  0000 C CNN
+F 1 "STM32F407VGTx" H 2650 820 50  0000 C CNN
+F 2 "Package_QFP:LQFP-100_14x14mm_P0.5mm" H 1950 1200 50  0001 R CNN
+F 3 "http://www.st.com/st-web-ui/static/active/en/resource/technical/document/datasheet/DM00037051.pdf" H 2650 3800 50  0001 C CNN
+	1    2650 3800
+	1    0    0    -1
+$EndComp
+$Comp
+L ina239-q1:INA239-Q1 U?
+U 1 1 6150C194
+P 5150 3550
+F 0 "U?" H 5150 3515 50  0000 C CNN
+F 1 "INA239-Q1" H 5150 3424 50  0000 C CNN
+F 2 "" H 5150 3550 50  0001 C CNN
+F 3 "" H 5150 3550 50  0001 C CNN
+	1    5150 3550
+	1    0    0    -1
+$EndComp
+$Comp
+L micro_sd_card_adafruit:Micro_SD_Card_Adafruit J?
+U 1 1 61515836
+P 6100 2450
+F 0 "J?" H 5700 3200 50  0000 L CNN
+F 1 "Micro_SD_Card_Adafruit" H 5950 3200 50  0000 L CNN
+F 2 "" H 8150 3150 50  0001 C CNN
+F 3 "https://www.hirose.com/product/en/download_file/key_name/DM3/category/Catalog/doc_file_id/49662/?file_category_id=4&item_id=195&is_series=1" H 6100 2550 50  0001 C CNN
+	1    6100 2450
+	1    0    0    -1
+$EndComp
 $EndSCHEMATC

Commit message: for report
Parts:
- removed U?: INA239-Q1, symbol ina239-q1:INA239-Q1
Changed lines of the file:
@@
-$EndComp
-$Comp
-L ina239-q1:INA239-Q1 U?
-U 1 1 6150C194
-P 5150 3550
-F 0 "U?" H 5150 3515 50  0000 C CNN
-F 1 "INA239-Q1" H 5150 3424 50  0000 C CNN
-F 2 "" H 5150 3550 50  0001 C CNN
-F 3 "" H 5150 3550 50  0001 C CNN
-	1    5150 3550
-	1    0    0    -1
 $EndComp
 $Comp
